Commit message: Updates to get the robot working in simulation

File: robomaster_description/urdf/alternate/arm.urdf.xacro (robot description, xacro)
@@ -240,5 +240,5 @@
         <origin xyz="0.1417841 0.0321051 -0.1257179" rpy="0 0 0"/>
         <mass value="0.009"/>
-        <inertia ixx="0.0205056" ixy="0.0021202" ixz="-0.0023248" iyy="0.0097562" iyz="0.0101162" izz="0.0117256"/>
+        <inertia ixx="0.1" ixy="0.0" ixz="0.0" iyy="0.1" iyz="0.0" izz="0.1"/>
       </inertial>
       <visual name="triangle">
@@ -256,23 +256,18 @@
       </collision>
     </link>
-    <joint name="${tf_prefix}arm_1_joint" type="revolute">
+    <joint name="${tf_prefix}arm_1_joint" type="fixed">
       <origin xyz="0.0103961 -0.0255713 0.030741" rpy="0 0 0"/>
       <parent link="${tf_prefix}arm_base_link"/>
       <child link="${tf_prefix}arm_1_link"/>
-      <axis xyz="0.0 1.0 0"/>
-      <limit effort="0" velocity="0" lower="-0.274" upper="1.384"/>
-    </joint>
-    <!-- <joint name="arm_2_dummy" type="floating">
+    </joint>
+    <!-- <joint name="arm_2_dummy" type="fixed">
       <origin xyz="-0.0419304 0.0028425 0.0218356" rpy="0 0 0"/>
       <parent link="arm_2_link"/>
       <child link="arm_2_dummy"/>
     </joint> -->
-    <joint name="${tf_prefix}arm_2_joint" type="continuous">
+    <joint name="${tf_prefix}arm_2_joint" type="fixed">
       <origin xyz="0.0018704 0.0438659 0.1210238" rpy="0 0 0"/>
       <parent link="${tf_prefix}arm_1_link"/>
       <child link="${tf_prefix}arm_2_link"/>
-      <axis xyz="0.0 1.0 0"/>
-      <limit effort="0" velocity="0"/>
-      <mimic joint="${tf_prefix}rod_3_joint" multiplier="-1.0" offset="0.0"/>
     </joint>
     <!-- <joint name="arm_base_attachment_joint" type="fixed">
@@ -286,5 +281,5 @@
       <child link="${tf_prefix}arm_base_link"/>
     </joint>
-    <!-- <joint name="attachement_link" type="floating">
+    <!-- <joint name="attachement_link" type="fixed">
       <origin xyz="0 0 0" rpy="0 0 0"/>
       <parent link="arm_base_link"/>
@@ -296,73 +291,58 @@
       <child link="${tf_prefix}end_point_link"/>
     </joint>
-    <joint name="${tf_prefix}endpoint_bracket_joint" type="continuous">
+    <joint name="${tf_prefix}endpoint_bracket_joint" type="fixed">
       <origin xyz="0.1058557 0.006752 -0.0561093" rpy="0 0 0"/>
       <parent link="${tf_prefix}arm_2_link"/>
       <child link="${tf_prefix}endpoint_bracket_link"/>
-      <axis xyz="0.0 1.0 0"/>
-      <mimic joint="${tf_prefix}rod_joint" multiplier="-1.0" offset="0.0"/>
-      <!-- <limit effort="0" velocity="0"/> -->
-    </joint>
-    <!-- <joint name="rod_1_dummy" type="floating">
+    </joint>
+    <!-- <joint name="rod_1_dummy" type="fixed">
       <origin xyz="-0.1048751 0 0.0582511" rpy="0 0 0"/>
       <parent link="rod_1_link"/>
       <child link="rod_1_dummy"/>
     </joint> -->
-    <joint name="${tf_prefix}rod_1_joint" type="continuous">
+    <joint name="${tf_prefix}rod_1_joint" type="fixed">
       <origin xyz="0.0134583 -0.0540971 0.0213068" rpy="0 -0.021293 0"/>
       <parent link="${tf_prefix}endpoint_bracket_link"/>
       <child link="${tf_prefix}rod_1_link"/>
-      <axis xyz="0.0 1.0 0"/>
-      <mimic joint="${tf_prefix}rod_joint" multiplier="1.0" offset="0.0"/>
-      <!-- <limit effort="0" velocity="0"/> -->
-    </joint>
-    <!-- <joint name="rod_2_dummy" type="floating">
+    </joint>
+    <!-- <joint name="rod_2_dummy" type="fixed">
       <origin xyz="0.0036225 0 0.1198535" rpy="0 0 0"/>
       <parent link="rod_2_link"/>
       <child link="rod_2_dummy"/>
     </joint> -->
-    <joint name="${tf_prefix}rod_2_joint" type="continuous">
+    <joint name="${tf_prefix}rod_2_joint" type="fixed">
       <origin xyz="-0.0224276 -0.0290701 0.0554782" rpy="0 -0.0094248 0"/>
       <parent link="${tf_prefix}arm_base_link"/>
       <child link="${tf_prefix}rod_2_link"/>
-      <axis xyz="0.0 1.0 0"/>
-      <mimic joint="${tf_prefix}arm_1_joint" multiplier="1.0" offset="0.0"/>
-      <!-- <limit effort="0" velocity="0"/> -->
-    </joint>
-    <!-- <joint name="rod_3_dummy" type="floating">
+    </joint>
+    <!-- <joint name="rod_3_dummy" type="fixed">
       <origin xyz="0.0029281 -0.0007404 0.1193638" rpy="0 0 0"/>
       <parent link="rod_3_link"/>
       <child link="rod_3_dummy"/>
     </joint> -->
-    <joint name="${tf_prefix}rod_3_joint" type="revolute">
+    <joint name="${tf_prefix}rod_3_joint" type="fixed">
       <origin xyz="-0.042397 0.0004533 0.0223131" rpy="0 0 0"/>
       <parent link="${tf_prefix}rod_link"/>
       <child link="${tf_prefix}rod_3_link"/>
-      <axis xyz="0.0 1.0 0"/>
-      <limit effort="0" velocity="0" lower="-0.34732" upper="1.21475"/>
-    </joint>
-    <joint name="${tf_prefix}rod_joint" type="revolute">
+    </joint>
+    <joint name="${tf_prefix}rod_joint" type="fixed">
       <origin xyz="0.009805 0.0214241 0.0319234" rpy="0 0 0"/>
       <parent link="${tf_prefix}arm_base_link"/>
       <child link="${tf_prefix}rod_link"/>
-      <axis xyz="0.0 1.0 0"/>
-      <limit effort="0" velocity="0" lower="-0.79936" upper="1.73137"/>
-    </joint>
-    <!-- <joint name="triangle_1_dummy" type="floating">
+    </joint>
+    <!-- <joint name="triangle_1_dummy" type="fixed">
       <origin xyz="-0.037193 0 0.0147539" rpy="0 0 0"/>
       <parent link="triangle_link"/>
       <child link="triangle_1_dummy"/>
     </joint> -->
-    <!-- <joint name="triangle_2_dummy" type="floating">
+    <!-- <joint name="triangle_2_dummy" type="fixed">
       <origin xyz="0.0077464 6.66e-05 0.0235099" rpy="0 0 0"/>
       <parent link="triangle_link"/>
       <child link="triangle_2_dummy"/>
     </joint> -->
-    <joint name="${tf_prefix}triangle_joint" type="continuous">
+    <joint name="${tf_prefix}triangle_joint" type="fixed">
       <origin xyz="0.0020224 -0.007103 0.1212334" rpy="0 0.2502802 0"/>
       <parent link="${tf_prefix}arm_1_link"/>
       <child link="${tf_prefix}triangle_link"/>
-      <axis xyz="0.0 1.0 0"/>
-      <mimic joint="${tf_prefix}arm_1_joint" multiplier="-1.0" offset="0.0"/>
     </joint>
     </xacro:macro>

File: robomaster_description/urdf/alternate/gripper.urdf.xacro (robot description, xacro)
@@ -144,13 +144,21 @@
         </link>
       <link name="${tf_prefix}gripper_m_link">
+        <inertial>
+          <origin xyz="0 0 0" rpy="0 0 0"/>
+          <mass value="0.001"/>
+          <inertia ixx="0.001" ixy="0" ixz="0" iyy="0.001" iyz="0" izz="0.001"/>
+        </inertial>
       </link>
       <link name="${tf_prefix}gripper_t_link">
+        <inertial>
+          <origin xyz="0 0 0" rpy="0 0 0"/>
+          <mass value="0.001"/>
+          <inertia ixx="0.001" ixy="0" ixz="0" iyy="0.001" iyz="0" izz="0.001"/>
+        </inertial>
       </link>
-      <joint name="${tf_prefix}gripper_m_joint" type="prismatic">
-        <limit effort="0" velocity="0" lower="-0.023" upper="0.001"/>
+      <joint name="${tf_prefix}gripper_m_joint" type="fixed">
         <origin xyz="0 0 0" rpy="0 0 0"/>
         <parent link="${tf_prefix}gripper_link_link"/>
         <child link="${tf_prefix}gripper_m_link"/>
-        <axis xyz="-1 0 0"/>
       </joint>
         <!-- <link name="left_gripper_8_link_dummy">
@@ -289,17 +297,13 @@
           </inertial>
         </link> -->
-        <joint name="${tf_prefix}left_gripper_joint_1" type="continuous">
+        <joint name="${tf_prefix}left_gripper_joint_1" type="fixed">
           <origin xyz="0.0163032 0.0212032 -0.0399201" rpy="0 0 0"/>
           <parent link="${tf_prefix}gripper_m_link"/>
           <child link="${tf_prefix}left_gripper_link_1"/>
-          <axis xyz="0 0 1.0"/>
-          <limit effort="0" velocity="0"/>
-        </joint>
-        <joint name="${tf_prefix}left_gripper_joint_2" type="continuous">
+        </joint>
+        <joint name="${tf_prefix}left_gripper_joint_2" type="fixed">
           <origin xyz="0.0213495 0.0130363 0" rpy="0 0 0"/>
           <parent link="${tf_prefix}left_gripper_link_1"/>
           <child link="${tf_prefix}left_gripper_link_2"/>
-          <axis xyz="0 0 1.0"/>
-          <limit effort="0" velocity="0"/>
         </joint>
         <!-- <joint name="left_gripper_joint_3_dummy" type="fixed">
@@ -308,24 +312,18 @@
           <child link="left_gripper_link_3_dummy"/>
         </joint> -->
-        <joint name="${tf_prefix}left_gripper_joint_4" type="continuous">
+        <joint name="${tf_prefix}left_gripper_joint_4" type="fixed">
           <origin xyz="0.00485 0.0204148 -5.8e-06" rpy="0 0 0"/>
           <parent link="${tf_prefix}left_gripper_link_2"/>
           <child link="${tf_prefix}left_gripper_link_4"/>
-          <axis xyz="0 0 1.0"/>
-          <limit effort="0" velocity="0"/>
-        </joint>
-        <joint name="${tf_prefix}left_gripper_joint_6" type="continuous">
+        </joint>
+        <joint name="${tf_prefix}left_gripper_joint_6" type="fixed">
           <origin xyz="0.0051144 -0.0140851 0" rpy="0 0 0"/>
           <parent link="${tf_prefix}left_gripper_link_5"/>
           <child link="${tf_prefix}left_gripper_link_6"/>
-          <axis xyz="0 0 1.0"/>
-          <limit effort="0" velocity="0"/>
-        </joint>
-        <joint name="${tf_prefix}left_gripper_joint_7" type="continuous">
+        </joint>
+        <joint name="${tf_prefix}left_gripper_joint_7" type="fixed">
           <origin xyz="-0.0148823 -0.0168513 0" rpy="0 0 0"/>
           <parent link="${tf_prefix}left_gripper_link_6"/>
           <child link="${tf_prefix}left_gripper_link_7"/>
-          <axis xyz="0 0 1.0"/>
-          <limit effort="0" velocity="0"/>
         </joint>
         <!-- <joint name="left_gripper_joint_8_dummy" type="fixed">
@@ -334,10 +332,8 @@
           <child link="left_gripper_8_link_dummy"/>
         </joint> -->
-        <joint name="${tf_prefix}left_gripper_joint_5" type="continuous">
+        <joint name="${tf_prefix}left_gripper_joint_5" type="fixed">
           <origin xyz="0.0385916 0.0103143 1.6e-06" rpy="0 0 0"/>
           <parent link="${tf_prefix}left_gripper_link_4"/>
           <child link="${tf_prefix}left_gripper_link_5"/>
-          <axis xyz="0 0 1.0"/>
-          <limit effort="0" velocity="0"/>
         </joint>
         <joint name="${tf_prefix}gripper_link" type="fixed">
@@ -346,17 +342,13 @@
           <child link="${tf_prefix}gripper_link_link"/>
         </joint>
-        <joint name="${tf_prefix}right_gripper_joint_1" type="continuous">
+        <joint name="${tf_prefix}right_gripper_joint_1" type="fixed">
           <origin xyz="0.0163034 -0.0209781 -0.0399201" rpy="0 0 0"/>
           <parent link="${tf_prefix}gripper_m_link"/>
           <child link="${tf_prefix}right_gripper_link_1"/>
-          <axis xyz="0 0 1.0"/>
-          <limit effort="0" velocity="0"/>
-        </joint>
-        <joint name="${tf_prefix}right_gripper_joint_2" type="continuous">
+        </joint>
+        <joint name="${tf_prefix}right_gripper_joint_2" type="fixed">
           <origin xyz="0.0213495 -0.0130363 0" rpy="0 0 0"/>
           <parent link="${tf_prefix}right_gripper_link_1"/>
           <child link="${tf_prefix}right_gripper_link_2"/>
-          <axis xyz="0 0 1.0"/>
-          <limit effort="0" velocity="0"/>
         </joint>
         <!-- <joint name="right_gripper_joint_3_dummy" type="fixed">
@@ -365,31 +357,23 @@
           <child link="right_gripper_link_3_dummy"/>
         </joint> -->
-        <joint name="${tf_prefix}right_gripper_joint_4" type="continuous">
+        <joint name="${tf_prefix}right_gripper_joint_4" type="fixed">
           <origin xyz="0.0047151 -0.0208481 -5.8e-06" rpy="0 0 0"/>
           <parent link="${tf_prefix}right_gripper_link_2"/>
           <child link="${tf_prefix}right_gripper_link_4"/>
-          <axis xyz="0 0 1.0"/>
-          <limit effort="0" velocity="0"/>
-        </joint>
-        <joint name="${tf_prefix}right_gripper_joint_5" type="continuous">
+        </joint>
+        <joint name="${tf_prefix}right_gripper_joint_5" type="fixed">
           <origin xyz="0.0385916 -0.0103143 1.6e-06" rpy="0 0 0"/>
           <parent link="${tf_prefix}right_gripper_link_4"/>
           <child link="${tf_prefix}right_gripper_link_5"/>
-          <axis xyz="0 0 1.0"/>
-          <limit effort="0" velocity="0"/>
-        </joint>
-        <joint name="${tf_prefix}right_gripper_joint_6" type="continuous">
+        </joint>
+        <joint name="${tf_prefix}right_gripper_joint_6" type="fixed">
           <origin xyz="0.0059278 0.0133069 0" rpy="0 0 0"/>
           <parent link="${tf_prefix}right_gripper_link_5"/>
           <child link="${tf_prefix}right_gripper_link_6"/>
-          <axis xyz="0 0 1.0"/>
-          <limit effort="0" velocity="0"/>
-        </joint>
-        <joint name="${tf_prefix}right_gripper_joint_7" type="continuous">
+        </joint>
+        <joint name="${tf_prefix}right_gripper_joint_7" type="fixed">
           <origin xyz="-0.0156955 0.0176295 0" rpy="0 0 0"/>
           <parent link="${tf_prefix}right_gripper_link_6"/>
           <child link="${tf_prefix}right_gripper_link_7"/>
-          <axis xyz="0 0 1.0"/>
-          <limit effort="0" velocity="0"/>
         </joint>
         <!-- <joint name="right_gripper_joint_8_dummy" type="fixed">

File: robomaster_description/urdf/base.urdf.xacro (robot description, xacro)
@@ -14,5 +14,5 @@
         <origin xyz="-0.0064553 -0.078141 0.0292877" rpy="0 0 0"/>
         <geometry>
-          <mesh filename="package://robomaster_description/meshes/armor.dae" scale="1.0 1.0 1.0"/>
+          <mesh filename="file:$(find robomaster_description)/meshes/armor.dae" scale="1.0 1.0 1.0"/>
         </geometry>
         <material name="armor_plastic"/>
@@ -21,5 +21,5 @@
         <origin xyz="-0.130336 -0.0018702 0.0174177" rpy="0 0 0"/>
         <geometry>
-          <mesh filename="package://robomaster_description/meshes/battery.dae" scale="1.0 1.0 1.0"/>
+          <mesh filename="file:$(find robomaster_description)/meshes/battery.dae" scale="1.0 1.0 1.0"/>
         </geometry>
         <material name="dark_plastic"/>
@@ -28,5 +28,5 @@
         <origin xyz="-0.1158907 0.066115 0.0525243" rpy="0 0 0"/>
         <geometry>
-          <mesh filename="package://robomaster_description/meshes/battery_pin_left.dae" scale="1.0 1.0 1.0"/>
+          <mesh filename="file:$(find robomaster_description)/meshes/battery_pin_left.dae" scale="1.0 1.0 1.0"/>
         </geometry>
         <material name="dark_plastic"/>
@@ -35,5 +35,5 @@
         <origin xyz="-0.1158907 -0.0658844 0.0525243" rpy="0 0 0"/>
         <geometry>
-          <mesh filename="package://robomaster_description/meshes/battery_pin_right.dae" scale="1.0 1.0 1.0"/>
+          <mesh filename="file:$(find robomaster_description)/meshes/battery_pin_right.dae" scale="1.0 1.0 1.0"/>
         </geometry>
         <material name="dark_plastic"/>
@@ -42,5 +42,5 @@
         <origin xyz="-0.0059039 0.0004154 0.0527955" rpy="0 0 0"/>
         <geometry>
-          <mesh filename="package://robomaster_description/meshes/chassis.dae" scale="1.0 1.0 1.0"/>
+          <mesh filename="file:$(find robomaster_description)/meshes/chassis.dae" scale="1.0 1.0 1.0"/>
         </geometry>
         <material name="chassis"/>
@@ -49,5 +49,5 @@
         <origin xyz="-0.1142288 -0.0006716 0.052675" rpy="0 0 0"/>
         <geometry>
-          <mesh filename="package://robomaster_description/meshes/controller.dae" scale="1.0 1.0 1.0"/>
+          <mesh filename="file:$(find robomaster_description)/meshes/controller.dae" scale="1.0 1.0 1.0"/>
         </geometry>
         <material name="dark_plastic"/>
@@ -56,5 +56,5 @@
         <origin xyz="-0.0787757 -0.002522 0.0720827" rpy="0 0 0"/>
         <geometry>
-          <mesh filename="package://robomaster_description/meshes/controller_cover.dae" scale="1.0 1.0 1.0"/>
+          <mesh filename="file:$(find robomaster_description)/meshes/controller_cover.dae" scale="1.0 1.0 1.0"/>
         </geometry>
         <material name="cover_plastic"/>
@@ -63,5 +63,5 @@
         <origin xyz="-0.0058789 -0.0001128 0.0294307" rpy="0 0 0"/>
         <geometry>
-          <mesh filename="package://robomaster_description/meshes/base_collision.dae" scale="1.0 1.0 1.0"/>
+          <mesh filename="file:$(find robomaster_description)/meshes/base_collision.dae" scale="1.0 1.0 1.0"/>
         </geometry>
       </collision>

File: robomaster_description/urdf/camera.urdf.xacro (robot description, xacro)
@@ -11,5 +11,5 @@
         <origin xyz="7.15e-05 0 -0.0004056" rpy="0 -1.7453293 0"/>
         <geometry>
-          <mesh filename="package://robomaster_description/meshes/camera.dae" scale="1.0 1.0 1.0000001"/>
+          <mesh filename="file:$(find robomaster_description)/meshes/camera.dae" scale="1.0 1.0 1.0000001"/>
         </geometry>
         <material name="metal"/>

File: robomaster_description/urdf/extension.urdf.xacro (robot description, xacro)
@@ -11,5 +11,5 @@
         <origin xyz="0 0 0" rpy="0 0 0"/>
         <geometry>
-          <mesh filename="package://robomaster_description/meshes/extension_base.dae" scale="1.0 1.0 1.0"/>
+          <mesh filename="file:$(find robomaster_description)/meshes/extension_base.dae" scale="1.0 1.0 1.0"/>
         </geometry>
         <material name="metal"/>
@@ -19,5 +19,5 @@
           <origin xyz="-0.078582 0.0075392 0.0046459" rpy="0 0 0"/>
           <geometry>
-            <mesh filename="package://robomaster_description/meshes/extension_support.dae" scale="1.0 1.0 1.0"/>
+            <mesh filename="file:$(find robomaster_description)/meshes/extension_support.dae" scale="1.0 1.0 1.0"/>
           </geometry>
           <material name="metal"/>
