Commit message: Updates to get the robot working in simulation

File: robomaster_description/urdf/gimbal.urdf.xacro (robot description, xacro)
@@ -11,5 +11,5 @@
         <origin xyz="0.00029 -0.03927 0.00764" rpy="0 0 0" />
         <geometry>
-          <mesh filename="package://robomaster_description/meshes/blaster_bug.dae" scale="0.7949 0.7949 0.7949" />
+          <mesh filename="file:$(find robomaster_description)/meshes/blaster_bug.dae" scale="0.7949 0.7949 0.7949" />
         </geometry>
         <material name="gimbal_armor" />
@@ -18,5 +18,5 @@
         <origin xyz="0.03896 0.00326 -0.01071" rpy="0 0 0" />
         <geometry>
-          <mesh filename="package://robomaster_description/meshes/blaster_gun.dae" scale="1.0 1.0 1.0" />
+          <mesh filename="file:$(find robomaster_description)/meshes/blaster_gun.dae" scale="1.0 1.0 1.0" />
         </geometry>
       </visual>
@@ -24,5 +24,5 @@
         <origin xyz="-0.02031 1e-05 0.02866" rpy="0 0 0" />
         <geometry>
-          <mesh filename="package://robomaster_description/meshes/blaster_magazin.dae" scale="1.0 1.0 1.0" />
+          <mesh filename="file:$(find robomaster_description)/meshes/blaster_magazin.dae" scale="1.0 1.0 1.0" />
         </geometry>
         <material name="plastic" />
@@ -31,5 +31,5 @@
         <origin xyz="0.0014 0.00082 0.01703" rpy="0 0 0"/>
         <geometry>
-          <mesh filename="package://robomaster_description/meshes/blaster_top.dae" scale="1.0 1.0 1.0" />
+          <mesh filename="file:$(find robomaster_description)/meshes/blaster_top.dae" scale="1.0 1.0 1.0" />
         </geometry>
         <material name="gimbal_top" />
@@ -38,5 +38,5 @@
         <origin xyz="0.03675 0.00135 -0.01024" rpy="0 0 0" />
         <geometry>
-          <mesh filename="package://robomaster_description/meshes/blaster_gun_collision.dae" scale="1.0 1.0 1.0" />
+          <mesh filename="file:$(find robomaster_description)/meshes/blaster_gun_collision.dae" scale="1.0 1.0 1.0" />
         </geometry>
       </collision>
@@ -44,5 +44,5 @@
         <origin xyz="-0.02168 1e-05 0.02911" rpy="0 0 0" />
         <geometry>
-          <mesh filename="package://robomaster_description/meshes/blaster_magazin_collision.dae" scale="1.0 1.0 1.0" />
+          <mesh filename="file:$(find robomaster_description)/meshes/blaster_magazin_collision.dae" scale="1.0 1.0 1.0" />
         </geometry>
       </collision>
@@ -50,5 +50,5 @@
         <origin xyz="0.00347 0.0008 0.01134" rpy="0 0 0" />
         <geometry>
-          <mesh filename="package://robomaster_description/meshes/blaster_top_collision.dae" scale="1.0 1.0 1.0" />
+          <mesh filename="file:$(find robomaster_description)/meshes/blaster_top_collision.dae" scale="1.0 1.0 1.0" />
         </geometry>
       </collision>
@@ -63,5 +63,5 @@
         <origin xyz="0 0 0" rpy="0 0 0" />
         <geometry>
-          <mesh filename="package://robomaster_description/meshes/gimbal_base.dae" scale="1.0 1.0 1.0" />
+          <mesh filename="file:$(find robomaster_description)/meshes/gimbal_base.dae" scale="1.0 1.0 1.0" />
         </geometry>
         <material name="gimbal" />
@@ -70,5 +70,5 @@
         <origin xyz="-0.00116 -0.00092 -0.00243" rpy="0 0 0" />
         <geometry>
-          <mesh filename="package://robomaster_description/meshes/gimbal_base_collision.dae" scale="1.0 1.0 1.0" />
+          <mesh filename="file:$(find robomaster_description)/meshes/gimbal_base_collision.dae" scale="1.0 1.0 1.0" />
         </geometry>
       </collision>
@@ -78,5 +78,5 @@
         <origin xyz="-0.02463 0 0.01615" rpy="0 0 0" />
         <geometry>
-          <mesh filename="package://robomaster_description/meshes/gimbal_left_led.dae" scale="1.0 1.0 1.0" />
+          <mesh filename="file:$(find robomaster_description)/meshes/gimbal_left_led.dae" scale="1.0 1.0 1.0" />
         </geometry>
         <material name="led_off" />
@@ -85,5 +85,5 @@
         <origin xyz="-0.02365 0 -0.01734" rpy="0 0 0"/>
         <geometry>
-          <mesh filename="package://robomaster_description/meshes/gimbal_left_led_0.dae" scale="1.0 1.0 1.0"/>
+          <mesh filename="file:$(find robomaster_description)/meshes/gimbal_left_led_0.dae" scale="1.0 1.0 1.0"/>
         </geometry>
         <material name="led_off"/>
@@ -92,5 +92,5 @@
         <origin xyz="-0.00837 0 -0.02777" rpy="0 0 0"/>
         <geometry>
-          <mesh filename="package://robomaster_description/meshes/gimbal_left_led_1.dae" scale="1.0 1.0 1.0"/>
+          <mesh filename="file:$(find robomaster_description)/meshes/gimbal_left_led_1.dae" scale="1.0 1.0 1.0"/>
         </geometry>
         <material name="led_off"/>
@@ -99,5 +99,5 @@
         <origin xyz="0.01027 0 -0.02687" rpy="0 0 0"/>
         <geometry>
-          <mesh filename="package://robomaster_description/meshes/gimbal_left_led_2.dae" scale="1.0 1.0 1.0"/>
+          <mesh filename="file:$(find robomaster_description)/meshes/gimbal_left_led_2.dae" scale="1.0 1.0 1.0"/>
         </geometry>
         <material name="led_off"/>
@@ -106,5 +106,5 @@
         <origin xyz="0.02428 0 -0.01501" rpy="0 0 0"/>
         <geometry>
-          <mesh filename="package://robomaster_description/meshes/gimbal_left_led_3.dae" scale="1.0 1.0 1.0"/>
+          <mesh filename="file:$(find robomaster_description)/meshes/gimbal_left_led_3.dae" scale="1.0 1.0 1.0"/>
         </geometry>
         <material name="led_off"/>
@@ -113,5 +113,5 @@
         <origin xyz="0.02289 -4e-05 0.01672" rpy="0 0 0"/>
         <geometry>
-          <mesh filename="package://robomaster_description/meshes/gimbal_left_led_4.dae" scale="1.0 1.0 1.0"/>
+          <mesh filename="file:$(find robomaster_description)/meshes/gimbal_left_led_4.dae" scale="1.0 1.0 1.0"/>
         </geometry>
         <material name="led_off"/>
@@ -120,5 +120,5 @@
         <origin xyz="0.00874 0 0.02703" rpy="0 0 0"/>
         <geometry>
-          <mesh filename="package://robomaster_description/meshes/gimbal_left_led_5.dae" scale="1.0 1.0 1.0"/>
+          <mesh filename="file:$(find robomaster_description)/meshes/gimbal_left_led_5.dae" scale="1.0 1.0 1.0"/>
         </geometry>
         <material name="led_off"/>
@@ -127,5 +127,5 @@
         <origin xyz="-0.00951 1e-05 0.02709" rpy="0 0 0"/>
         <geometry>
-          <mesh filename="package://robomaster_description/meshes/gimbal_left_led_6.dae" scale="1.0 1.0 1.0"/>
+          <mesh filename="file:$(find robomaster_description)/meshes/gimbal_left_led_6.dae" scale="1.0 1.0 1.0"/>
         </geometry>
         <material name="led_off"/>
@@ -134,5 +134,5 @@
         <origin xyz="-0.02463 0 0.01615" rpy="0 0 0"/>
         <geometry>
-          <mesh filename="package://robomaster_description/meshes/gimbal_left_led_7.dae" scale="1.0 1.0 1.0"/>
+          <mesh filename="file:$(find robomaster_description)/meshes/gimbal_left_led_7.dae" scale="1.0 1.0 1.0"/>
         </geometry>
         <material name="led_off"/>
@@ -143,5 +143,5 @@
         <origin xyz="-0.02364 -9e-05 -0.01734" rpy="0 0 0"/>
         <geometry>
-          <mesh filename="package://robomaster_description/meshes/gimbal_right_led_0.dae" scale="1.0 1.0 1.0"/>
+          <mesh filename="file:$(find robomaster_description)/meshes/gimbal_right_led_0.dae" scale="1.0 1.0 1.0"/>
         </geometry>
         <material name="led_off"/>
@@ -150,5 +150,5 @@
         <origin xyz="-0.00837 -0.00011 -0.02778" rpy="0 0 0"/>
         <geometry>
-          <mesh filename="package://robomaster_description/meshes/gimbal_right_led_1.dae" scale="1.0 1.0 1.0"/>
+          <mesh filename="file:$(find robomaster_description)/meshes/gimbal_right_led_1.dae" scale="1.0 1.0 1.0"/>
         </geometry>
         <material name="led_off"/>
@@ -157,5 +157,5 @@
         <origin xyz="0.01027 -0.00011 -0.02687" rpy="0 0 0"/>
         <geometry>
-          <mesh filename="package://robomaster_description/meshes/gimbal_right_led_2.dae" scale="1.0 1.0 1.0"/>
+          <mesh filename="file:$(find robomaster_description)/meshes/gimbal_right_led_2.dae" scale="1.0 1.0 1.0"/>
         </geometry>
         <material name="led_off"/>
@@ -164,5 +164,5 @@
         <origin xyz="0.02428 -0.00011 -0.01501" rpy="0 0 0"/>
         <geometry>
-          <mesh filename="package://robomaster_description/meshes/gimbal_right_led_3.dae" scale="1.0 1.0 1.0"/>
+          <mesh filename="file:$(find robomaster_description)/meshes/gimbal_right_led_3.dae" scale="1.0 1.0 1.0"/>
         </geometry>
         <material name="led_off"/>
@@ -171,5 +171,5 @@
         <origin xyz="0.0229 0.00017 0.01671" rpy="0 0 0"/>
         <geometry>
-          <mesh filename="package://robomaster_description/meshes/gimbal_right_led_4.dae" scale="1.0 1.0 1.0"/>
+          <mesh filename="file:$(find robomaster_description)/meshes/gimbal_right_led_4.dae" scale="1.0 1.0 1.0"/>
         </geometry>
         <material name="led_off"/>
@@ -178,5 +178,5 @@
         <origin xyz="0.00874 8e-05 0.02709" rpy="0 0 0"/>
         <geometry>
-          <mesh filename="package://robomaster_description/meshes/gimbal_right_led_5.dae" scale="1.0 1.0 1.0"/>
+          <mesh filename="file:$(find robomaster_description)/meshes/gimbal_right_led_5.dae" scale="1.0 1.0 1.0"/>
         </geometry>
         <material name="led_off"/>
@@ -185,5 +185,5 @@
         <origin xyz="-0.00957 8e-05 0.02706" rpy="0 0 0"/>
         <geometry>
-          <mesh filename="package://robomaster_description/meshes/gimbal_right_led_6.dae" scale="1.0 1.0 1.0"/>
+          <mesh filename="file:$(find robomaster_description)/meshes/gimbal_right_led_6.dae" scale="1.0 1.0 1.0"/>
         </geometry>
         <material name="led_off"/>
@@ -192,5 +192,5 @@
         <origin xyz="-0.02463 8e-05 0.01615" rpy="0 0 0"/>
         <geometry>
-          <mesh filename="package://robomaster_description/meshes/gimbal_right_led7.dae" scale="1.0 1.0 1.0"/>
+          <mesh filename="file:$(find robomaster_description)/meshes/gimbal_right_led7.dae" scale="1.0 1.0 1.0"/>
         </geometry>
         <material name="led_off"/>
@@ -206,5 +206,5 @@
         <origin xyz="-2e-05 -0.001 0.03369" rpy="0 0 0" />
         <geometry>
-          <mesh filename="package://robomaster_description/meshes/gimbal.dae" scale="1.0 1.0 1.0" />
+          <mesh filename="file:$(find robomaster_description)/meshes/gimbal.dae" scale="1.0 1.0 1.0" />
         </geometry>
         <material name="gimbal" />
@@ -213,5 +213,5 @@
         <origin xyz="-0.00472 0.06418 0.07122" rpy="0 0 0" />
         <geometry>
-          <mesh filename="package://robomaster_description/meshes/gimbal_left_armor.dae" scale="1.0 1.0 1.0" />
+          <mesh filename="file:$(find robomaster_description)/meshes/gimbal_left_armor.dae" scale="1.0 1.0 1.0" />
         </geometry>
         <material name="gimbal_armor" />
@@ -220,5 +220,5 @@
         <origin xyz="-0.00527 -0.06277 0.07314" rpy="0 0 0" />
         <geometry>
-          <mesh filename="package://robomaster_description/meshes/gimbal_right_armor.dae" scale="1.0 1.0 1.0" />
+          <mesh filename="file:$(find robomaster_description)/meshes/gimbal_right_armor.dae" scale="1.0 1.0 1.0" />
         </geometry>
         <material name="gimbal_armor" />
@@ -227,5 +227,5 @@
         <origin xyz="-0.00027 0.00034 0.08755" rpy="0 0 0" />
         <geometry>
-          <mesh filename="package://robomaster_description/meshes/gimbal_side.dae" scale="1.0 1.0 1.0" />
+          <mesh filename="file:$(find robomaster_description)/meshes/gimbal_side.dae" scale="1.0 1.0 1.0" />
         </geometry>
         <material name="gimbal_side" />
@@ -234,5 +234,5 @@
         <origin xyz="-0.01647 -0.05644 0.05429" rpy="0 0 0" />
         <geometry>
-          <mesh filename="package://robomaster_description/meshes/gimbal_collision.dae" scale="1.0 1.0 1.0" />
+          <mesh filename="file:$(find robomaster_description)/meshes/gimbal_collision.dae" scale="1.0 1.0 1.0" />
         </geometry>
       </collision>
@@ -247,5 +247,5 @@
         <origin xyz="0 0 0" rpy="0 0 0" />
         <geometry>
-          <mesh filename="package://robomaster_description/meshes/speaker.dae" scale="1.0 1.0 1.0" />
+          <mesh filename="file:$(find robomaster_description)/meshes/speaker.dae" scale="1.0 1.0 1.0" />
         </geometry>
         <material name="Material #32.001" />
@@ -254,5 +254,5 @@
         <origin xyz="-0.00408 -0.00356 -0.00071" rpy="0 0 0" />
         <geometry>
-          <mesh filename="package://robomaster_description/meshes/speaker_collision.dae" scale="1.0 1.0 1.0" />
+          <mesh filename="file:$(find robomaster_description)/meshes/speaker_collision.dae" scale="1.0 1.0 1.0" />
         </geometry>
       </collision>

File: robomaster_description/urdf/intelligent_controller.urdf.xacro (robot description, xacro)
@@ -11,5 +11,5 @@
         <origin xyz="0 0 -0.0095231" rpy="0 0 0"/>
         <geometry>
-          <mesh filename="package://robomaster_description/meshes/intelligent_controller.dae" scale="1.0 1.0 1.0"/>
+          <mesh filename="file:$(find robomaster_description)/meshes/intelligent_controller.dae" scale="1.0 1.0 1.0"/>
         </geometry>
         <material name="intelligent_controller"/>
@@ -18,5 +18,5 @@
         <origin xyz="-0.0147105 0.0344787 0.0032872" rpy="0 0 0"/>
         <geometry>
-          <mesh filename="package://robomaster_description/meshes/wifi_antenna_left.dae" scale="1.0 1.0 1.0"/>
+          <mesh filename="file:$(find robomaster_description)/meshes/wifi_antenna_left.dae" scale="1.0 1.0 1.0"/>
         </geometry>
         <material name="intelligent_controller"/>
@@ -25,5 +25,5 @@
         <origin xyz="-0.0147125 -0.0351398 0.0042003" rpy="0 0 0"/>
         <geometry>
-          <mesh filename="package://robomaster_description/meshes/wifi_antenna_right.dae" scale="1.0 1.0 1.0"/>
+          <mesh filename="file:$(find robomaster_description)/meshes/wifi_antenna_right.dae" scale="1.0 1.0 1.0"/>
         </geometry>
         <material name="intelligent_controller"/>

File: robomaster_description/urdf/led.urdf.xacro (robot description, xacro)
@@ -11,5 +11,5 @@
       <origin xyz="0 0 0" rpy="0 0 0"/>
       <geometry>
-        <mesh filename="package://robomaster_description/meshes/hit_sensor.dae" scale="1.0 1.0 1.0"/>
+        <mesh filename="file:$(find robomaster_description)/meshes/hit_sensor.dae" scale="1.0 1.0 1.0"/>
       </geometry>
       <material name="hit_detector"/>
@@ -25,5 +25,5 @@
       <origin xyz="0 0 0" rpy="0 0 0"/>
       <geometry>
-        <mesh filename="package://robomaster_description/meshes/led.dae" scale="1.0 1.0 1.0"/>
+        <mesh filename="file:$(find robomaster_description)/meshes/led.dae" scale="1.0 1.0 1.0"/>
       </geometry>
       <material name="led_light"/>

File: robomaster_description/urdf/wheel.urdf.xacro (robot description, xacro)
@@ -1,4 +1,4 @@
 <?xml version="1.0"?>
-<robot xmlns:xacro="http://playerstage.sourceforge.net/gazebo/xmlschema/#xacro">
+<robot xmlns:xacro="http://playerstage.sourceforge.net/gazebo/xmlschema/#xacro" xmlns:ignition="http://gazebosim.org/schema">
   <xacro:macro name="wheel" params="name xyz direction side tf_prefix=''">
     <link name="${tf_prefix}${name}_wheel_link">
@@ -20,18 +20,28 @@
         <origin xyz="0 0 0" rpy="0 0 0"/>
         <geometry>
-          <mesh filename="package://robomaster_description/meshes/wheel.dae" scale="1.0 ${direction} 1.0"/>
+          <mesh filename="file:$(find robomaster_description)/meshes/wheel.dae" scale="1.0 ${direction} 1.0"/>
         </geometry>
         <material name="wheel_plastic"/>
       </visual>
-      <collision name="${name}_wheel">
+      <collision>
         <origin xyz="0 0 0" rpy="${pi/2} 0 0"/>
         <geometry>
           <cylinder radius="0.05" length="0.042"/>
         </geometry>
-        <material name="collision">
-          <color rgba="0.8 0.0 0.0 1.0"/>
-        </material>
       </collision>
     </link>
+    <gazebo reference='${tf_prefix}${name}_wheel_link'>
+      <collision>
+        <surface>
+          <friction>
+            <ode>
+              <mu>1.0</mu>
+              <mu2>0.0</mu2>
+              <fdir1 ignition:expressed_in="base_link">1 ${-1.0 * direction} 0</fdir1>
+            </ode>
+          </friction>
+        </surface>
+      </collision>
+    </gazebo>
     <joint name="${tf_prefix}${name}_wheel_joint" type="continuous">
       <origin xyz="${xyz}" rpy="0 0 0"/>
@@ -39,5 +49,4 @@
       <child link="${tf_prefix}${name}_wheel_link"/>
       <axis xyz="0 1.0 0"/>
-      <limit effort="0" velocity="0"/>
     </joint>
   </xacro:macro>
