Commit message: Make wheel collision cylinders shorter to make the simulation match more closely the kinetic model

File: robomaster_description/urdf/wheel.urdf.xacro (robot description, xacro)
@@ -27,5 +27,5 @@
         <origin xyz="0 0 0" rpy="${pi/2} 0 0"/>
         <geometry>
-          <cylinder radius="0.05" length="0.042"/>
+          <cylinder radius="0.05" length="0.005"/>
         </geometry>
       </collision>
